Commit message: Gazebo Simulation

File: urdf/delivery_bot.urdf (robot description, URDF)
Before this commit: robot delivery_bot, 4 links, 3 joints
Links:
- link left_wheel_link: mass None -> 1.0; geometry collision cylinder length=0.03 radius=0.07; visual cylinder length=0.03 radius=0.07
- link lidar_link: mass None -> 0.5; geometry collision cylinder length=0.05 radius=0.05; visual cylinder length=0.05 radius=0.05
- link right_wheel_link: mass None -> 1.0; geometry collision cylinder length=0.03 radius=0.07; visual cylinder length=0.03 radius=0.07
Joints:
- joint left_wheel_joint: axis (none) -> 0 1 0; type fixed -> continuous
- joint right_wheel_joint: axis (none) -> 0 1 0; type fixed -> continuous

Commit message: New updates

File: urdf/delivery_bot.urdf (robot description, URDF)
Before this commit: robot delivery_bot, 4 links, 3 joints
Joints:
- joint left_wheel_joint: origin xyz=0 0.18 0.05 rpy=0 0 0 -> xyz=0 0.18 0.0 rpy=0 0 0
- joint lidar_joint: origin xyz=0 0 0.15 rpy=0 0 0 -> xyz=0 0 0.30 rpy=0 0 0
- joint right_wheel_joint: origin xyz=0 -0.18 0.05 rpy=0 0 0 -> xyz=0 -0.18 0.0 rpy=0 0 0
